File: USB HUB.kicad_pcb (KiCad board)
At the start: 2 copper layers, 30 x 91.8 mm, 15 parts, among them J1 USB3_A, J2 USB3_A, J3 USB3_A, J4 USB3_A, J5 Conn_01x09_Socket, U1 FE1.1s, Y1 Crystal_GND24

Commit message: just saved file
Parts:
- moved U1 64.2 mm to (190.2, 28.4), turned to -90 degrees
- moved R1 30.2 mm to (134.0, 55.3), turned to -90 degrees
